Commit message: MoveIt! Namespaces may be working

File: src/my_abb_irb120/config/abb_irb120_3_58_macro.srdf.xacro (robot description, xacro)
@@ -4,5 +4,6 @@
     A URDF file must exist for this robot as well, where the joints and the links that are referenced are defined
 -->
-<robot name="abb_irb120_3_58">
+<robot xmlns:xacro="http://ros.org/wiki/xacro">
+<xacro:macro name="abb_irb120_3_58_g" params="prefix robotns">
     <!--GROUPS: Representation of a set of joints and links. This can be useful for specifying DOF to plan for, defining arms, end effectors, etc-->
     <!--LINKS: When a link is specified, the parent joint of that link (if it exists) is automatically included-->
@@ -10,9 +11,9 @@
     <!--CHAINS: When a chain is specified, all the links along the chain (including endpoints) are included in the group. Additionally, all the joints that are parents to included links are also included. This means that joints along the chain and the parent joint of the base link are included in the group-->
     <!--SUBGROUPS: Groups can also be formed by referencing to already defined group names-->
-    <group name="manipulator">
+    <group name="${robotns}/manipulator">
         <chain base_link="base_link" tip_link="tool0" />
     </group>
     <!--GROUP STATES: Purpose: Define a named state for a particular group, in terms of joint values. This is useful to define states like 'folded arms'-->
-    <group_state name="all_zero" group="manipulator">
+    <group_state name="all_zero" group="${robotns}/manipulator">
         <joint name="joint_1" value="0" />
         <joint name="joint_2" value="0" />
@@ -37,3 +38,4 @@
     <disable_collisions link1="link_4" link2="link_6" reason="Default" />
     <disable_collisions link1="link_5" link2="link_6" reason="Adjacent" />
+  </xacro:macro>
 </robot>
