Commit message: Fixed Gazebo's namespaces

File: src/my_abb_irb120/urdf/irb120_3_58.xacro (robot description, xacro)
@@ -2,5 +2,5 @@
 <robot name="abb_irb120_3_58" xmlns:xacro="http://ros.org/wiki/xacro">
   <xacro:include filename="$(find my_abb_irb120)/urdf/irb120_3_58_macro.xacro"/>
-  <xacro:abb_irb120_3_58_g prefix="" robotname=""/>
+  <xacro:abb_irb120_3_58_g prefix="" robotns=""/>
   <!-- Fix robot to Gazebo world -->
   <link name="world"/>

File: src/my_abb_irb120/urdf/irb120_3_58_macro.xacro (robot description, xacro)
@@ -2,7 +2,7 @@
 <robot xmlns:xacro="http://ros.org/wiki/xacro">
 <xacro:include filename="$(find my_abb_irb120)/urdf/irb120_3_58_support_macro.xacro"/>
-<xacro:macro name="abb_irb120_3_58_g" params="prefix robotname">
+<xacro:macro name="abb_irb120_3_58_g" params="prefix robotns">
   <!-- get base ABB IRB120 model -->
-  <xacro:abb_irb120_3_58 prefix="${prefix}" robotname="${robotname}"/>
+  <xacro:abb_irb120_3_58 prefix="${prefix}" robotns="${robotns}"/>
   <!-- transmission list -->
   <transmission name="${prefix}tran1">
@@ -93,5 +93,5 @@
   <gazebo>
     <plugin name="gazebo_ros_control" filename="libgazebo_ros_control.so">
-      <robotNamespace>${robotname}</robotNamespace>
+      <robotnsspace>${robotns}</robotnsspace>
       <robotSimType>gazebo_ros_control/DefaultRobotHWSim</robotSimType>
     </plugin>

File: src/my_abb_irb120/urdf/irb120_3_58_support_macro.xacro (robot description, xacro)
@@ -2,5 +2,5 @@
 <robot xmlns:xacro="http://ros.org/wiki/xacro">
   <xacro:include filename="$(find abb_resources)/urdf/common_materials.xacro"/>
-  <xacro:macro name="abb_irb120_3_58" params="prefix robotname">
+  <xacro:macro name="abb_irb120_3_58" params="prefix robotns">
     <!-- link list -->
     <link name="${prefix}base_link">

Commit message: Namespace C++ integration

File: src/my_abb_irb120/urdf/irb120_3_58.xacro (robot description, xacro)
@@ -1,11 +1,13 @@
 <?xml version="1.0" ?>
 <robot name="abb_irb120_3_58" xmlns:xacro="http://ros.org/wiki/xacro">
+  <xacro:arg name="prefix" default="" />
+  <xacro:arg name="robotns" default="" />
   <xacro:include filename="$(find my_abb_irb120)/urdf/irb120_3_58_macro.xacro"/>
-  <xacro:abb_irb120_3_58_g prefix="" robotns=""/>
+  <xacro:abb_irb120_3_58_g prefix="$(arg prefix)" robotns="$(arg robotns)"/>
   <!-- Fix robot to Gazebo world -->
   <link name="world"/>
   <joint name="world-base_link-fixed" type="fixed">
     <parent link="world"/>
-    <child link="base_link"/>
+    <child link="$(arg prefix)base_link"/>
   </joint>
 </robot>
