Commit message: Changed values to radians in pose

File: src/multiple_abb_irb120/config/abb_irb120_3_58_macro.srdf.xacro (robot description, xacro)
@@ -25,8 +25,8 @@
     <group_state name="demo_pose" group="${robotns}_manipulator">
         <joint name="joint_1" value="0" />
-        <joint name="joint_2" value="12" />
-        <joint name="joint_3" value="-6" />
+        <joint name="joint_2" value="0.21" />
+        <joint name="joint_3" value="-0.1" />
         <joint name="joint_4" value="0" />
-        <joint name="joint_5" value="84" />
+        <joint name="joint_5" value="1.466" />
         <joint name="joint_6" value="0" />
     </group_state>

Commit message: MoveIt Planning Safety
Spheres creation in Planning Scene
Tool link added

File: src/multiple_abb_irb120/config/abb_irb120_3_58_macro.srdf.xacro (robot description, xacro)
@@ -12,5 +12,5 @@
     <!--SUBGROUPS: Groups can also be formed by referencing to already defined group names-->
     <group name="${robotns}_manipulator">
-        <chain base_link="base_link" tip_link="tool0" />
+        <chain base_link="base_link" tip_link="tool_link" />
     </group>
     <!--GROUP STATES: Purpose: Define a named state for a particular group, in terms of joint values. This is useful to define states like 'folded arms'-->

File: src/multiple_abb_irb120/urdf/irb120_3_58_with_tool.xacro (robot description, xacro)
@@ -11,3 +11,12 @@
     <child link="$(arg prefix)base_link"/>
   </joint>
+  <!-- Add an imaginary tool for planning with MoveIt -->
+  <link name="$(arg prefix)tool_link">
+    <origin xyz="0 0 0" rpy="0 0 0"/>
+  </link>
+  <joint name="$(arg prefix)tool_joint" type="fixed">
+    <origin xyz="0 0 0.075" rpy="0 0 0"/>
+    <parent link="$(arg prefix)tool0"/>
+    <child link="$(arg prefix)tool_link"/>
+  </joint>
 </robot>

Commit message: Todo horrible

File: src/multiple_abb_irb120/config/abb_irb120_3_58_macro.srdf.xacro (robot description, xacro)
@@ -12,38 +12,38 @@
     <!--SUBGROUPS: Groups can also be formed by referencing to already defined group names-->
     <group name="${robotns}_manipulator">
-        <chain base_link="base_link" tip_link="tool_link" />
+        <chain base_link="${robotns}_base_link" tip_link="${robotns}_tool_link" />
     </group>
     <!--GROUP STATES: Purpose: Define a named state for a particular group, in terms of joint values. This is useful to define states like 'folded arms'-->
     <group_state name="all_zero" group="${robotns}_manipulator">
-        <joint name="joint_1" value="0" />
-        <joint name="joint_2" value="0" />
-        <joint name="joint_3" value="0" />
-        <joint name="joint_4" value="0" />
-        <joint name="joint_5" value="0" />
-        <joint name="joint_6" value="0" />
+        <joint name="${robotns}_joint_1" value="0" />
+        <joint name="${robotns}_joint_2" value="0" />
+        <joint name="${robotns}_joint_3" value="0" />
+        <joint name="${robotns}_joint_4" value="0" />
+        <joint name="${robotns}_joint_5" value="0" />
+        <joint name="${robotns}_joint_6" value="0" />
     </group_state>
     <group_state name="demo_pose" group="${robotns}_manipulator">
-        <joint name="joint_1" value="0" />
-        <joint name="joint_2" value="0.21" />
-        <joint name="joint_3" value="-0.1" />
-        <joint name="joint_4" value="0" />
-        <joint name="joint_5" value="1.466" />
-        <joint name="joint_6" value="0" />
+        <joint name="${robotns}_joint_1" value="0" />
+        <joint name="${robotns}_joint_2" value="0.21" />
+        <joint name="${robotns}_joint_3" value="-0.1" />
+        <joint name="${robotns}_joint_4" value="0" />
+        <joint name="${robotns}_joint_5" value="1.466" />
+        <joint name="${robotns}_joint_6" value="0" />
     </group_state>
     <!--VIRTUAL JOINT: Purpose: this element defines a virtual joint between a robot link and an external frame of reference (considered fixed with respect to the robot)-->
-    <virtual_joint name="FixedBase" type="fixed" parent_frame="world" child_link="base_link" />
+    <virtual_joint name="FixedBase" type="fixed" parent_frame="world" child_link="${robotns}_base_link" />
     <!--DISABLE COLLISIONS: By default it is assumed that any link of the robot could potentially come into collision with any other link in the robot. This tag disables collision checking between a specified pair of links. -->
-    <disable_collisions link1="base_link" link2="link_1" reason="Adjacent" />
-    <disable_collisions link1="base_link" link2="link_2" reason="Never" />
-    <disable_collisions link1="link_1" link2="link_2" reason="Adjacent" />
-    <disable_collisions link1="link_2" link2="link_3" reason="Adjacent" />
-    <disable_collisions link1="link_2" link2="link_5" reason="Never" />
-    <disable_collisions link1="link_2" link2="link_6" reason="Never" />
-    <disable_collisions link1="link_3" link2="link_4" reason="Adjacent" />
-    <disable_collisions link1="link_3" link2="link_5" reason="Never" />
-    <disable_collisions link1="link_3" link2="link_6" reason="Never" />
-    <disable_collisions link1="link_4" link2="link_5" reason="Adjacent" />
-    <disable_collisions link1="link_4" link2="link_6" reason="Default" />
-    <disable_collisions link1="link_5" link2="link_6" reason="Adjacent" />
+    <disable_collisions link1="${robotns}_base_link" link2="${robotns}_link_1" reason="Adjacent" />
+    <disable_collisions link1="${robotns}_base_link" link2="${robotns}_link_2" reason="Never" />
+    <disable_collisions link1="${robotns}_link_1" link2="${robotns}_link_2" reason="Adjacent" />
+    <disable_collisions link1="${robotns}_link_2" link2="${robotns}_link_3" reason="Adjacent" />
+    <disable_collisions link1="${robotns}_link_2" link2="${robotns}_link_5" reason="Never" />
+    <disable_collisions link1="${robotns}_link_2" link2="${robotns}_link_6" reason="Never" />
+    <disable_collisions link1="${robotns}_link_3" link2="${robotns}_link_4" reason="Adjacent" />
+    <disable_collisions link1="${robotns}_link_3" link2="${robotns}_link_5" reason="Never" />
+    <disable_collisions link1="${robotns}_link_3" link2="${robotns}_link_6" reason="Never" />
+    <disable_collisions link1="${robotns}_link_4" link2="${robotns}_link_5" reason="Adjacent" />
+    <disable_collisions link1="${robotns}_link_4" link2="${robotns}_link_6" reason="Default" />
+    <disable_collisions link1="${robotns}_link_5" link2="${robotns}_link_6" reason="Adjacent" />
   </xacro:macro>
 </robot>
