Commit message: Changed package name and added RobotInterface

File: src/multiple_abb_irb120/config/abb_irb120_3_58.srdf.xacro (robot description, xacro)
@@ -3,5 +3,5 @@
   <xacro:arg name="prefix" default="robot1_" />
   <xacro:arg name="robotns" default="robot1" />
-  <xacro:include filename="$(find my_abb_irb120)/config/abb_irb120_3_58_macro.srdf.xacro"/>
+  <xacro:include filename="$(find multiple_abb_irb120)/config/abb_irb120_3_58_macro.srdf.xacro"/>
   <xacro:abb_irb120_3_58_g prefix="$(arg prefix)" robotns="$(arg robotns)"/>
 </robot>

File: src/multiple_abb_irb120/config/abb_irb120_3_58_macro.srdf.xacro (robot description, xacro)
@@ -23,4 +23,12 @@
         <joint name="joint_6" value="0" />
     </group_state>
+    <group_state name="demo_pose" group="${robotns}/manipulator">
+        <joint name="joint_1" value="0" />
+        <joint name="joint_2" value="12" />
+        <joint name="joint_3" value="-6" />
+        <joint name="joint_4" value="0" />
+        <joint name="joint_5" value="84" />
+        <joint name="joint_6" value="0" />
+    </group_state>
     <!--VIRTUAL JOINT: Purpose: this element defines a virtual joint between a robot link and an external frame of reference (considered fixed with respect to the robot)-->
     <virtual_joint name="FixedBase" type="fixed" parent_frame="world" child_link="base_link" />

File: src/multiple_abb_irb120/urdf/irb120_3_58.xacro (robot description, xacro)
@@ -3,5 +3,5 @@
   <xacro:arg name="prefix" default="" />
   <xacro:arg name="robotns" default="" />
-  <xacro:include filename="$(find my_abb_irb120)/urdf/irb120_3_58_macro.xacro"/>
+  <xacro:include filename="$(find multiple_abb_irb120)/urdf/irb120_3_58_macro.xacro"/>
   <xacro:abb_irb120_3_58_g prefix="$(arg prefix)" robotns="$(arg robotns)"/>
   <!-- Fix robot to Gazebo world -->

File: src/multiple_abb_irb120/urdf/irb120_3_58_macro.xacro (robot description, xacro)
@@ -1,5 +1,5 @@
 <?xml version="1.0"?>
 <robot xmlns:xacro="http://ros.org/wiki/xacro">
-<xacro:include filename="$(find my_abb_irb120)/urdf/irb120_3_58_support_macro.xacro"/>
+<xacro:include filename="$(find multiple_abb_irb120)/urdf/irb120_3_58_support_macro.xacro"/>
 <xacro:macro name="abb_irb120_3_58_g" params="prefix robotns">
   <!-- get base ABB IRB120 model -->

Commit message: Fixed move_group and MoveGroupInterface connections
Now move_group node connects to the adequate joint_states topic
MoveGroupInterface connects to the adequate joint_states topic (robot names must be unique)

File: src/multiple_abb_irb120/config/abb_irb120_3_58.srdf.xacro (robot description, xacro)
@@ -1,5 +1,5 @@
 <?xml version="1.0" ?>
-<robot name="abb_irb120_3_58" xmlns:xacro="http://ros.org/wiki/xacro">
-  <xacro:arg name="prefix" default="robot1_" />
+<robot name="abb_irb120_3_58_$(arg robotns)" xmlns:xacro="http://ros.org/wiki/xacro">
+  <xacro:arg name="prefix" default="" />
   <xacro:arg name="robotns" default="robot1" />
   <xacro:include filename="$(find multiple_abb_irb120)/config/abb_irb120_3_58_macro.srdf.xacro"/>

File: src/multiple_abb_irb120/urdf/irb120_3_58_with_tool.xacro (robot description, xacro)
@@ -1,8 +1,8 @@
 <?xml version="1.0" ?>
-<robot name="abb_irb120_3_58" xmlns:xacro="http://ros.org/wiki/xacro">
+<robot name="abb_irb120_3_58_$(arg robotns)" xmlns:xacro="http://ros.org/wiki/xacro">
   <xacro:arg name="prefix" default="" />
-  <xacro:arg name="robotns" default="" />
+  <xacro:arg name="robotns" default="robot1" />
   <xacro:include filename="$(find multiple_abb_irb120)/urdf/irb120_3_58_macro.xacro"/>
-  <xacro:abb_irb120_3_58_g prefix="$(arg prefix)" robotns="$(arg robotns)"/>
+  <xacro:abb_irb120_3_58_g prefix="$(arg prefix)" robotns="/$(arg robotns)"/>
   <!-- Fix robot to Gazebo world -->
   <link name="world"/>
@@ -12,5 +12,5 @@
   </joint>
   <!-- Add an imaginary tool for planning with MoveIt -->
-  <link name="$(arg prefix)tool_link">
+  <link name="tool_link">
     <origin xyz="0 0 0" rpy="0 0 0"/>
   </link>
@@ -18,5 +18,5 @@
     <origin xyz="0 0 0.075" rpy="0 0 0"/>
     <parent link="$(arg prefix)tool0"/>
-    <child link="$(arg prefix)tool_link"/>
+    <child link="tool_link"/>
   </joint>
 </robot>
